File: mcr_shield.kicad_pcb (KiCad board)
At the start: 2 copper layers, 135 x 95 mm, 23 parts, among them J2 MCR_P1_Controls, J3 MCR_System_Coin, J4 MCR_Opt_X_Dial, J5 MCR_P2_Controls, SW1 Game_Selector, SW2 Cabinet_Options, U1 Buck_Regulator, U2 Optocoupler_P1, U3 Optocoupler_Sys, U4 Sync_Buffer, U5 Audio_Amplifier

Commit message: routed
Routing:
- net GND: track 0.00 -> 320.5 mm
- net BTN_LEFT: track 0.00 -> 92.2 mm
- net BTN_RIGHT: track 0.00 -> 84.1 mm
- net BTN_FIRE: track 0.00 -> 82.3 mm
- net BTN_SHIELD: track 0.00 -> 74.3 mm
- net FPGA_R1: track 0.00 -> 71.1 mm, vias 0 -> 1
- net FPGA_R0: track 0.00 -> 66.3 mm
- net FPGA_R2: track 0.00 -> 65.1 mm, vias 0 -> 1
- net SPINNER_D7: track 0.00 -> 60.9 mm
- net CAB_P2_LEFT: track 0.00 -> 60.2 mm
- net SPINNER_D6: track 0.00 -> 58.4 mm
- net CAB_P2_RIGHT: track 0.00 -> 57.6 mm
- net CAB_P2_FIRE: track 0.00 -> 55.1 mm
- net 5V_REGULATED: track 0.00 -> 53.8 mm
- net FPGA_G0: track 0.00 -> 53.5 mm
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