File: MCR_prototype_PCB/MCR_prototype_PCB.kicad_pcb (KiCad board)
At the start: 2 copper layers, 266.7 x 203.2 mm, 210 parts, among them J0 Conn_02x20_Odd_Even, J1 Conn_01x20_Pin, J1-VGAOut1 DE15_Socket_HighDensity, J2_RGBS_Out1 Conn_01x09_Pin, J3 Conn_01x09_Pin, J4 Conn_01x19_Pin, J5 Conn_01x23_Pin, J6 Conn_01x10_Pin, SW1 SW_DIP_x08, SW2 SW_DIP_x08, U1 74AHC165, U10 ULN2803CDWR, U11 ULN2803CDWR, U12 THS7374, U13 THS7374, U14 ADS7830, U2 74AHC165, U20 LM2596T-5, U21 LM2596T-3.3, U3 74AHC165, U4 74AHC165, U6 74AHC165, U7 74AHC165, U8 74HC595, U9 74HC595

Commit message: Updated 8/22/26
Parts:
- removed C6, C8: 220 uF, Capacitor_THT:CP_Radial_D8.0mm_P3.50mm
- removed D10, D11, D12, D13, D14, D15, D16, D17, D18, D19, D20, D21, D22, D23, D24, D25, D26, D27, D28, D29, D30, D31, D32, D33, D34, D4, D5, D6, D7, D8, D9: BAT54S, Package_TO_SOT_SMD:SOT-23
- removed R12, R13, R14, R15, R16, R17, R18, R19, R20, R21, R33, R35, R37, R39, R41, R43, R45, R47, R49, R51, R53, R55, R57, R59, R61, R63, R65, R67, R69, R71, R73, R75, R76, R77, R78, R79, R80, R81, R82, R83, R84, R85, R86, R87, R88, R89, R90, R91: 4.7k, Resistor_SMD:R_0805_2012Metric
- removed R22, R23, R24, R25, R26, R27, R28, R29, R30, R31, R32, R34, R36, R38, R40, R42, R44, R46, R48, R50, R52, R54, R56, R58, R60, R62, R64, R66, R68, R70, R72, R74: 1k, Resistor_SMD:R_0805_2012Metric
- removed U20: LM2596T-5, Package_TO_SOT_THT:TO-220-5_P3.4x3.7mm_StaggerOdd_Lead3.8mm_Vertical
- removed U21: LM2596T-3.3, Package_TO_SOT_THT:TO-220-5_P3.4x3.7mm_StaggerOdd_Lead3.8mm_Vertical
- added R6: 2k ohm, Resistor_SMD:R_0805_2012Metric_Pad1.20x1.40mm_HandSolder, F.Cu at (96.7, 128.2)
- added R7: 510 ohm, Resistor_SMD:R_0805_2012Metric_Pad1.20x1.40mm_HandSolder, F.Cu at (97.1, 97.4)
- added R8: 220 ohm, Resistor_SMD:R_0805_2012Metric_Pad1.20x1.40mm_HandSolder, F.Cu at (96.9, 113.8)
- added RN1: 4.7k ohm, Resistor_THT:R_Array_SIP9, F.Cu at (225.9, 199.0)
- added RN10: 1K Ohm, Resistor_SMD:R_Array_Convex_4x0603, F.Cu at (263.1, 165.0)
- added RN11: 1K Ohm, Resistor_SMD:R_Array_Convex_4x0603, F.Cu at (261.1, 63.2)
- added RN12: 1K Ohm, Resistor_SMD:R_Array_Convex_4x0603, F.Cu at (261.6, 71.8)
- added RN13: 1K Ohm, Resistor_SMD:R_Array_Convex_4x0603, F.Cu at (262.4, 131.8)
- added RN14: 1K Ohm, Resistor_SMD:R_Array_Convex_4x0603, F.Cu at (262.4, 117.1)
- added RN2: 4.7k ohm, Resistor_THT:R_Array_SIP9, F.Cu at (226.1, 169.2)
- added RN3: 4.7k ohm, Resistor_THT:R_Array_SIP9, F.Cu at (226.0, 77.5)
- added RN4: 4.7k ohm, Resistor_THT:R_Array_SIP9, F.Cu at (226.5, 134.1)
- added RN5: 4.7k ohm, Resistor_THT:R_Array_SIP9, F.Cu at (112.4, 53.1)
- added RN6: 4.7k ohm, Resistor_THT:R_Array_SIP9, F.Cu at (112.0, 81.0)
- added RN7: 1K Ohm, Resistor_SMD:R_Array_Convex_4x0603, F.Cu at (262.4, 186.6)
- added RN8: 1K Ohm, Resistor_SMD:R_Array_Convex_4x0603, F.Cu at (262.8, 197.6)
- added RN9: 1K Ohm, Resistor_SMD:R_Array_Convex_4x0603, F.Cu at (263.0, 153.2)
- added U15: SRV05-4, Package_TO_SOT_SMD:SOT-23-6, F.Cu at (250.5, 151.1)
- added U16: SRV05-4, Package_TO_SOT_SMD:SOT-23-6, F.Cu at (238.3, 181.5)
- added U17: SRV05-4, Package_TO_SOT_SMD:SOT-23-6, F.Cu at (247.5, 181.6)
- added U18: SRV05-4, Package_TO_SOT_SMD:SOT-23-6, F.Cu at (238.4, 56.6)
- added U19: SRV05-4, Package_TO_SOT_SMD:SOT-23-6, F.Cu at (250.6, 56.6)
- added U22: SRV05-4, Package_TO_SOT_SMD:SOT-23-6, F.Cu at (243.9, 116.0)
- added U23: SRV05-4, Package_TO_SOT_SMD:SOT-23-6, F.Cu at (252.3, 116.1)
- added U24: R-78B5.0-2.0, Converter_DCDC:Converter_DCDC_RECOM_R-78B-2.0_THT, F.Cu at (77.1, 97.6)
- added U25: R-78B3.3-2.0, Converter_DCDC:Converter_DCDC_RECOM_R-78B-2.0_THT, F.Cu at (77.3, 113.9)
- added U5: SRV05-4, Package_TO_SOT_SMD:SOT-23-6, F.Cu at (241.5, 150.7)
- C5, C7: value 680 uF -> 4.7 uF 50V
- D1, D2: value 1N5824 -> LED; footprint Diode_THT:D_DO-201AD_P15.24mm_Horizontal -> LED_SMD:LED_0805_2012Metric_Pad1.15x1.40mm_HandSolder
- D3: value BAT54S -> LED; footprint Package_TO_SOT_SMD:SOT-23 -> LED_SMD:LED_0805_2012Metric_Pad1.15x1.40mm_HandSolder
- D35, D36, D37, D38: footprint LED_SMD:LED_0805_2012Metric -> LED_SMD:LED_0805_2012Metric_Pad1.15x1.40mm_HandSolder
- L1, L2: value 33 uH -> 3.3 uH
- R101, R95, R98: value 1000 -> 1k
- R102, R96, R99: value 2000 -> 2k
- moved D3 159.1 mm to (92.2, 114.0)
- moved U10 97.1 mm to (234.3, 22.7)
- moved U8 96.8 mm to (221.0, 23.4)
- moved U9 93.1 mm to (221.1, 39.9)
- moved U11 93.1 mm to (234.5, 39.3)
- moved C33 62.0 mm to (239.2, 124.1), turned to 90 degrees
- moved C34 56.8 mm to (244.7, 124.1), turned to 90 degrees
- moved C17 56.2 mm to (237.7, 158.4), turned to 90 degrees
- moved U2 55.1 mm to (215.2, 158.9)
- moved C35 52.5 mm to (249.8, 124.4), turned to 90 degrees
- moved J0 51.8 mm to (125.2, 148.1), turned to 180 degrees
- moved C18 50.8 mm to (243.5, 158.4), turned to 90 degrees
- moved C36 48.1 mm to (254.7, 124.2), turned to 90 degrees
- moved C37 47.8 mm to (238.5, 129.9), turned to 90 degrees
- moved C16 47.4 mm to (252.9, 189.3), turned to 90 degrees
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Connections:
- C9 pad 2: Net-(D3-COM) -> Net-(U16-IO2)
- D1 pad 1: Net-(D1-K) -> GND
- D1 pad 2: GND -> Net-(D1-A)
- D2 pad 1: Net-(D2-K) -> GND
- D2 pad 2: GND -> Net-(D2-A)
- D3 pad 2: +5V -> Net-(D3-A)
- L1 pad 1: Net-(D1-K) -> +12V
- L1 pad 2: +5V -> Net-(U24-IN)
- L2 pad 1: Net-(D2-K) -> +12V
- L2 pad 2: +3.3V -> Net-(U25-IN)
Routing:
- net +5V: track 1055.1 -> 111.3 mm, vias 10 -> 15
- net GND: track 1193.8 -> 253.8 mm, vias 5 -> 35
- net VID_G2: track 79.2 -> 222.3 mm, vias 0 -> 2
- net +12V: track 223.3 -> 359.0 mm, vias 2 -> 3
- net SEL: track 150.5 -> 37.3 mm, vias 0 -> 1
- net Coin_Meter: track 153.3 -> 41.5 mm, vias 0 -> 1
- net Coin_Meter_Return: track 147.5 -> 36.5 mm, vias 0 -> 1
- net MD3: track 150.6 -> 40.0 mm
- net MD1: track 147.8 -> 40.0 mm, vias 2 -> 1
- net MD2: track 145.8 -> 43.1 mm, vias 2 -> 1
- net ST1: track 131.4 -> 34.1 mm
- net MD0: track 143.2 -> 48.4 mm
- net ARD: track 128.5 -> 38.2 mm, vias 0 -> 1
- net ST0: track 129.9 -> 46.7 mm
- net Out_Data: track 99.8 -> 170.0 mm, vias 3 -> 2
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- added copper zone on In2.Cu, net +5V
- added copper zone on In1.Cu, net GND
Other:
- board size 266.7 x 203.2 mm -> 267.1 x 198.7 mm
- copper layers 2 -> 4
- board text added: "+12V OK"
- board text added: "+3.3V OK"
- board text added: "+5V OK"
- board text added: "TANG 60K"

Commit message: Add files via upload
Parts:
- added C46: 0.01 uF, Capacitor_SMD:C_0805_2012Metric, F.Cu at (224.9, 97.1)
- added C47: 0.01 uF, Capacitor_SMD:C_0805_2012Metric, F.Cu at (224.8, 101.0)
- added C6: 0.01 uF, Capacitor_SMD:C_0805_2012Metric, F.Cu at (225.0, 90.1)
- added C8: 0.01 uF, Capacitor_SMD:C_0805_2012Metric, F.Cu at (224.9, 93.7)
- added D4: 1N4148W, Diode_SMD:D_SOD-123, F.Cu at (115.4, 132.8)
- added J3_DOT1: Conn_01x10_Pin, Mitch_Custom:PinHeader_1x10_P2.54mm_Horizontal_mirrored, F.Cu at (253.9, 83.4)
- added R10: 1k, Resistor_SMD:R_0805_2012Metric, F.Cu at (229.4, 90.0)
- added R11: 1k, Resistor_SMD:R_0805_2012Metric, F.Cu at (229.4, 93.6)
- added R12: 1k, Resistor_SMD:R_0805_2012Metric, F.Cu at (229.4, 97.2)
- added R13: 1k, Resistor_SMD:R_0805_2012Metric, F.Cu at (229.3, 101.0)
- added R9: 1k, Resistor_SMD:R_0805_2012Metric_Pad1.20x1.40mm_HandSolder, F.Cu at (115.2, 138.2)
- added SW4: Service, Button_Switch_SMD:SW_SPDT_CK_JS102011SAQN, F.Cu at (205.2, 23.7)
- added TP1: +12V Input, TestPoint:TestPoint_Loop_D1.80mm_Drill1.0mm_Beaded, F.Cu at (78.3, 126.6)
- added TP2: +3.3V Power, TestPoint:TestPoint_Loop_D1.80mm_Drill1.0mm_Beaded, F.Cu at (84.7, 109.0)
- added TP3: +5V Power, TestPoint:TestPoint_Loop_D1.80mm_Drill1.0mm_Beaded, F.Cu at (85.4, 91.6)
- added TP4: Gnd, TestPoint:TestPoint_Loop_D1.80mm_Drill1.0mm_Beaded, F.Cu at (77.9, 136.7)
- added TP5: In_Clk, TestPoint:TestPoint_Loop_D1.80mm_Drill1.0mm_Beaded, F.Cu at (104.9, 112.8)
- added TP6: IN_LOAD_N, TestPoint:TestPoint_Loop_D1.80mm_Drill1.0mm_Beaded, F.Cu at (108.1, 122.1)
- added TP7: VID_HS, TestPoint:TestPoint_Loop_D1.80mm_Drill1.0mm_Beaded, F.Cu at (191.7, 17.4)
- added TP8: VID_VS, TestPoint:TestPoint_Loop_D1.80mm_Drill1.0mm_Beaded, F.Cu at (192.0, 24.6)
- added TP9: GND, TestPoint:TestPoint_Loop_D1.80mm_Drill1.0mm_Beaded, F.Cu at (256.9, 142.1)
- moved R6 7.54 mm to (89.7, 130.9), turned to -90 degrees
- moved D1 6.94 mm to (89.7, 134.9), turned to 90 degrees
- moved C1 5.09 mm to (244.8, 87.5)
- moved C2 5.09 mm to (244.8, 92.5)
- moved C3 5.09 mm to (244.8, 98.0)
- moved C4 5.09 mm to (244.8, 103.0)
- moved C45 5.09 mm to (244.8, 108.0)
- moved R1 5.09 mm to (239.8, 87.5)
- moved R2 5.09 mm to (239.8, 92.7)
- moved R3 5.09 mm to (239.8, 98.0)
- moved R4 5.09 mm to (239.8, 103.1)
- moved R5 5.09 mm to (239.8, 108.0)
- moved U14 5.09 mm to (242.2, 81.0)
- moved D3 5.06 mm to (93.6, 118.9), turned to 90 degrees
- moved R7 4.53 mm to (92.6, 98.0), turned to -90 degrees
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Connections:
- net AUD_PWM_L renamed AUD_PWM_L1
- net AUD_PWM_R renamed AUD_PWM_R1
- net Net-(J5-Pin_1) renamed /1 Plyr Move Left
- net Net-(J5-Pin_2) renamed /1 Plyr Move Right
- net Net-(J5-Pin_3) renamed /1 Plyr Move Up
- net Net-(J5-Pin_4) renamed /1 Plyr Move Down
- J0 pad 1: unconnected-(J0-Pin_1-Pad1) -> AUD_PWM_L2
- J0 pad 11: unconnected-(J0-Pin_11-Pad11) -> Net-(D4-K)
- J0 pad 5: unconnected-(J0-Pin_5-Pad5) -> AUD_PWM_R2
- J0 pad 9: unconnected-(J0-Pin_9-Pad9) -> Service Switch
- J4 pad 19: unconnected-(J4-Pin_19-Pad19) -> GND
- J4 pad 9: unconnected-(J4-Pin_9-Pad9) -> GND
Routing:
- net Service Switch: track 0.00 -> 156.2 mm, vias 0 -> 3
- net AUD_PWM_L2: track 0.00 -> 139.0 mm, vias 0 -> 2
- net AUD_PWM_R2: track 0.00 -> 135.4 mm, vias 0 -> 2
- net GND: track 253.8 -> 380.4 mm, vias 35 -> 40
- net VID_G2: track 222.3 -> 106.8 mm, vias 2 -> 1
- net +5V: track 111.3 -> 191.2 mm
- net Net-(J3_DOT1-Pin_10): track 0.00 -> 36.8 mm, vias 0 -> 2
- net Out_Data: track 170.0 -> 135.4 mm, vias 2 -> 1
- net Net-(J3_DOT1-Pin_9): track 0.00 -> 33.6 mm, vias 0 -> 2
- net +3.3V: track 386.9 -> 419.4 mm, vias 10 -> 11
- net VID_R2: track 117.0 -> 146.8 mm, vias 2 -> 3
- net VID_R1: track 121.0 -> 150.7 mm
- net Net-(RN14-R4.2): track 86.3 -> 58.8 mm, vias 2 -> 3
- net LED_DDR_RST: track 78.7 -> 103.3 mm
- net Net-(RN6-R1): track 61.8 -> 39.5 mm
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
Commit message: Add files via upload
Parts:
- removed C10, C11, C12, C13, C14, C15, C16, C17, C18, C19, C20, C21, C22, C23, C24, C25, C26, C27, C28, C29, C30, C31, C32, C33, C34, C35, C36, C37, C38, C39, C40, C9: 0.01 uF, Capacitor_SMD:C_0805_2012Metric
- removed SW4: Service, Button_Switch_SMD:SW_SPDT_CK_JS102011SAQN
- added C48: 0.1 uF, Capacitor_SMD:C_0805_2012Metric, F.Cu at (88.0, 102.0)
- added C49: 100 uF, Capacitor_SMD:CP_Elec_6.3x5.4, F.Cu at (103.2, 100.2)
- added C50: 0.1 uF, Capacitor_SMD:C_0805_2012Metric, F.Cu at (89.0, 119.1)
- added C51: 100 uF, Capacitor_SMD:CP_Elec_6.3x5.4, F.Cu at (100.5, 118.9)
- added C52: 0.1 uF, Capacitor_SMD:C_0805_2012Metric, F.Cu at (215.4, 178.7)
- added C53: 0.1 uF, Capacitor_SMD:C_0805_2012Metric, F.Cu at (215.2, 149.5)
- added C54: 0.1 uF, Capacitor_SMD:C_0805_2012Metric, F.Cu at (205.5, 67.6)
- added C55: 0.1 uF, Capacitor_SMD:C_0805_2012Metric, F.Cu at (215.5, 132.6)
- added C56: 0.1 uF, Capacitor_SMD:C_0805_2012Metric, F.Cu at (103.1, 29.4)
- added C57: 0.1 uF, Capacitor_SMD:C_0805_2012Metric, F.Cu at (102.5, 63.0)
- added C58: 0.1 uF, Capacitor_SMD:C_0805_2012Metric, F.Cu at (214.5, 35.8)
- added C59: 0.1 uF, Capacitor_SMD:C_0805_2012Metric, F.Cu at (234.5, 79.2)
- added C60: 0.1 uF, Capacitor_SMD:C_0805_2012Metric, F.Cu at (215.2, 16.2)
- added C61: 0.1 uF, Capacitor_SMD:C_0805_2012Metric, F.Cu at (232.5, 53.9)
- added C62: 0.1 uF, Capacitor_SMD:C_0805_2012Metric, F.Cu at (255.6, 54.4)
- added C63: 0.1 uF, Capacitor_SMD:C_0805_2012Metric, F.Cu at (238.7, 116.2)
- added C64: 0.1 uF, Capacitor_SMD:C_0805_2012Metric, F.Cu at (252.8, 111.0)
- added JP4: VGA Filter, Connector_PinHeader_2.54mm:PinHeader_1x03_P2.54mm_Vertical, F.Cu at (125.4, 38.1)
- added R104: 10k, Resistor_SMD:R_0805_2012Metric, F.Cu at (214.5, 30.9)
- added R14: 75, Resistor_SMD:R_0805_2012Metric, F.Cu at (161.0, 32.0)
- added R15: 75, Resistor_SMD:R_0805_2012Metric, F.Cu at (165.5, 32.1)
- added R16: 75, Resistor_SMD:R_0805_2012Metric, F.Cu at (170.1, 32.1)
- added R17: 75, Resistor_SMD:R_0805_2012Metric, F.Cu at (174.5, 32.1)
- added R18: 75, Capacitor_SMD:C_0805_2012Metric, F.Cu at (179.8, 34.3)
- added SW3: Service, Button_Switch_SMD:SW_SPST_PTS645Sx43SMTR92, F.Cu at (205.6, 18.7)
- D4: value 1N4148W -> 1N5822; footprint Diode_SMD:D_SOD-123 -> Diode_THT:D_DO-201AD_P15.24mm_Horizontal
- moved TP1 20.4 mm to (57.9, 128.3)
- moved TP4 12.9 mm to (89.7, 141.9)
- moved JP3 2.35 mm to (61.3, 59.9)
Connections:
- J5 pad 18: unconnected-(J5-Pin_18-Pad18) -> GND
- J5 pad 21: Coin_Meter_Return -> +12V
- J5 pad 9: unconnected-(J5-Pin_9-Pad9) -> GND
- U1 pad 1: IN_CLK -> IN_LOAD_N
- U1 pad 2: IN_LOAD_N -> IN_CLK
- U10 pad 17: Coin_Meter_Return -> unconnected-(U10-O2-Pad17)
- U12 pad 13: Net-(J2_RGBS_Out1-Pin_9) -> Net-(U12-CH2_OUT)
- U12 pad 14: Net-(J2_RGBS_Out1-Pin_8) -> Net-(U12-CH1_OUT)
- U12 pad 9: GND -> Net-(JP4-C)
- U13 pad 12: Net-(J2_RGBS_Out1-Pin_3) -> Net-(U13-CH3_OUT)
- U13 pad 13: Net-(J2_RGBS_Out1-Pin_5) -> Net-(U13-CH2_OUT)
- U13 pad 14: Net-(J2_RGBS_Out1-Pin_1) -> Net-(U13-CH1_OUT)
- U13 pad 9: GND -> Net-(JP4-C)
- U14 pad 16: +3.3V -> +5V
- U15 pad 1: Net-(U15-IO1) -> Net-(RN2-R2)
- U15 pad 3: Net-(U15-IO2) -> Net-(RN2-R1)
- U15 pad 4: Net-(U15-IO3) -> Net-(RN2-R3)
- U15 pad 6: Net-(U15-IO4) -> Net-(RN2-R4)
- U16 pad 1: Net-(U16-IO1) -> Net-(RN1-R2)
- U16 pad 3: Net-(U16-IO2) -> Net-(RN1-R1)
- U16 pad 4: Net-(U16-IO3) -> Net-(RN1-R3)
- U16 pad 6: Net-(U16-IO4) -> Net-(RN1-R4)
- U17 pad 1: Net-(U17-IO1) -> Net-(RN1-R6)
- U17 pad 3: Net-(U17-IO2) -> Net-(RN1-R5)
- U17 pad 4: Net-(U17-IO3) -> Net-(RN1-R7)
- U17 pad 6: Net-(U17-IO4) -> Net-(RN1-R8)
- U18 pad 1: Net-(U18-IO1) -> Net-(RN11-R3.2)
- U18 pad 3: Net-(U18-IO2) -> Net-(RN11-R4.2)
- U18 pad 4: Net-(U18-IO3) -> Net-(RN11-R2.2)
- U18 pad 6: Net-(U18-IO4) -> Net-(RN11-R1.2)
- U19 pad 1: Net-(U19-IO1) -> Net-(RN12-R3.2)
- U19 pad 3: Net-(U19-IO2) -> Net-(RN12-R4.2)
- U19 pad 4: Net-(U19-IO3) -> Net-(RN12-R2.2)
- U19 pad 6: Net-(U19-IO4) -> Net-(RN12-R1.2)
- U2 pad 1: IN_CLK -> IN_LOAD_N
- U2 pad 2: IN_LOAD_N -> IN_CLK
- U22 pad 1: Net-(U22-IO1) -> Net-(RN14-R3.2)
- U22 pad 3: Net-(U22-IO2) -> Net-(RN14-R4.2)
- U22 pad 4: Net-(U22-IO3) -> Net-(RN14-R2.2)
- U22 pad 6: Net-(U22-IO4) -> Net-(RN14-R1.2)
- U23 pad 1: Net-(U23-IO1) -> Net-(RN13-R3.2)
- U23 pad 3: Net-(U23-IO2) -> Net-(RN13-R4.2)
- U23 pad 4: Net-(U23-IO3) -> Net-(RN13-R2.2)
- U23 pad 6: Net-(U23-IO4) -> Net-(RN13-R1.2)
- U5 pad 1: Net-(U5-IO1) -> Net-(RN10-R3.2)
- U5 pad 3: Net-(U5-IO2) -> Net-(RN10-R4.2)
- U5 pad 4: Net-(U5-IO3) -> Net-(RN10-R2.2)
- U5 pad 6: Net-(U5-IO4) -> Net-(RN10-R1.2)
Routing:
- net +5V: track 191.2 -> 316.3 mm, vias 15 -> 21
- net GND: track 380.4 -> 297.5 mm, vias 40 -> 41
- net Net-(JP4-C): track 0.00 -> 53.6 mm, vias 0 -> 2
- net +3.3V: track 419.4 -> 464.7 mm, vias 11 -> 13
- net Out_Data: track 135.4 -> 179.0 mm, vias 1 -> 2
- net +12V: track 356.5 -> 398.1 mm
- net Coin_Meter_Return: track 36.5 -> 0.00 mm, vias 1 -> 0
- net Net-(RN1-R2): track 54.1 -> 83.9 mm
- net IN_LOAD_N: track 310.7 -> 339.2 mm
- net VID_G2: track 106.8 -> 135.1 mm
- net Net-(U16-IO4): track 25.9 -> 0.00 mm, vias 2 -> 0
- net LED_PIX: track 110.8 -> 85.4 mm, vias 2 -> 1
- net VID_R2: track 146.8 -> 122.4 mm, vias 3 -> 1
- net Net-(U18-IO4): track 23.1 -> 0.00 mm, vias 2 -> 0
- net Net-(U19-IO1): track 22.0 -> 0.00 mm, vias 2 -> 0
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Other:
- board text added: "Filter Off"
- board text added: "Filter On"

Commit message: Add files via upload
Parts:
- added C10: 10 uF 50V, Capacitor_THT:CP_Radial_D10.0mm_P5.00mm, F.Cu at (62.8, 87.1)
- added C65: 0.1 uF, Capacitor_SMD:C_0805_2012Metric, F.Cu at (249.8, 82.7)
- added C9: 10 uF 50V, Capacitor_THT:CP_Radial_D10.0mm_P5.00mm, F.Cu at (72.2, 124.1)
- added R19: 75, Resistor_SMD:R_0805_2012Metric, F.Cu at (167.0, 56.3)
- added R20: 75, Resistor_SMD:R_0805_2012Metric, F.Cu at (174.5, 56.2)
- added R21: 75, Resistor_SMD:R_0805_2012Metric, F.Cu at (180.6, 56.2)
- added R22: 1k, Resistor_SMD:R_0805_2012Metric, F.Cu at (249.1, 77.5)
- added R23: 1k, Resistor_SMD:R_0805_2012Metric, F.Cu at (244.8, 76.5)
- added REFLL: MountingHole_4.3mm_M4, MountingHole:MountingHole_4.3mm_M4, F.Cu at (31.6, 182.0)
- added REFLM: MountingHole_4.3mm_M4, MountingHole:MountingHole_4.3mm_M4, F.Cu at (151.2, 169.7)
- added REFLR: MountingHole_4.3mm_M4, MountingHole:MountingHole_4.3mm_M4, F.Cu at (252.6, 173.5)
- added REFUL: MountingHole_4.3mm_M4, MountingHole:MountingHole_4.3mm_M4, F.Cu at (28.5, 44.6)
- added REFUR: MountingHole_4.3mm_M4, MountingHole:MountingHole_4.3mm_M4, F.Cu at (273.8, 11.1)
Connections:
- C59 pad 1: +5V -> +3.3V
- J3 pad 1: +5V -> +3.3V
- J3_DOT1 pad 1: +5V -> +3.3V
- J5 pad 20: Coin_Meter -> +12V
- J5 pad 21: +12V -> Coin_Meter
- U14 pad 10: +5V -> Net-(U14-REFin/REFout)
- U14 pad 16: +5V -> +3.3V
Routing:
- net +3.3V: track 464.7 -> 586.2 mm
- net GND: track 297.5 -> 323.8 mm, vias 41 -> 45
- net Net-(U24-IN): track 10.2 -> 27.5 mm
- net Net-(U25-IN): track 10.7 -> 21.1 mm
- net +12V: track 398.1 -> 408.0 mm
- net +5V: track 316.3 -> 307.4 mm, vias 21 -> 19
- net Net-(U13-CH3_IN): track 22.3 -> 28.0 mm
- net Net-(U13-CH1_IN): track 21.5 -> 27.2 mm
- net Net-(U13-CH2_IN): track 21.1 -> 26.7 mm
- net Net-(U14-REFin/REFout): track 0.00 -> 5.17 mm
- net ADC_SCL: track 142.1 -> 146.9 mm
- net ADC_SDA: track 162.0 -> 166.5 mm
- net Coin_Meter: track 41.5 -> 39.4 mm

Commit message: September 8 Version
Parts:
- removed REFLL, REFLM, REFLR, REFUL, REFUR: MountingHole_4.3mm_M4, MountingHole:MountingHole_4.3mm_M4
- L1, L2: value 3.3 uH -> FAUL1360-3R3MT
- SW1, SW2: value SW_DIP_x08 -> DSIC08LHGET
- SW3: value Service -> PTS645SM43SMTR92LFS
- U24: value R-78B5.0-2.0 -> K7805-2000R3
- U25: value R-78B3.3-2.0 -> K7803-2000R3
