File: MCR_prototype_PCB/MCR_prototype_PCB.kicad_pcb (KiCad board)
At the start: 4 copper layers, 267.1 x 198.7 mm, 143 parts, among them J0 Conn_02x20_Odd_Even, J1 Conn_01x20_Pin, J1-VGAOut1 DE15_Socket_HighDensity, J2_RGBS_Out1 Conn_01x09_Pin, J3 Conn_01x09_Pin, J3_DOT1 Conn_01x10_Pin, J4 Conn_01x19_Pin, J5 Conn_01x23_Pin, J6 Conn_01x10_Pin, SW1 DSIC08LHGET, SW2 DSIC08LHGET, SW3 PTS645SM43SMTR92LFS, U1 74AHC165, U10 ULN2803CDWR, U11 ULN2803CDWR, U12 THS7374, U13 THS7374, U14 ADS7830, U15 SRV05-4, U16 SRV05-4, U17 SRV05-4, U18 SRV05-4, U19 SRV05-4, U2 74AHC165, U22 SRV05-4, U23 SRV05-4, U24 K7805-2000R3, U25 K7803-2000R3, U3 74AHC165, U4 74AHC165, U5 SRV05-4, U6 74AHC165, U7 74AHC165, U8 74HC595, U9 74HC595

Commit message: Production/schematics for 10/10/26 first board run
Parts:
- added C66: 0.1 uF, Capacitor_SMD:C_0805_2012Metric, F.Cu at (248.4, 158.5)
- added C67: 0.1 uF, Capacitor_SMD:C_0805_2012Metric, F.Cu at (248.4, 170.7)
- added C68: 0.1 uF, Capacitor_SMD:C_0805_2012Metric, F.Cu at (248.8, 185.0)
- added C69: 0.1 uF, Capacitor_SMD:C_0805_2012Metric, F.Cu at (249.3, 198.3)
- C10, C9: footprint Capacitor_THT:CP_Radial_D10.0mm_P5.00mm -> Capacitor_SMD:CP_Elec_6.3x5.4
- C5, C7: footprint Capacitor_THT:CP_Radial_D10.0mm_P5.00mm -> Capacitor_SMD:CP_Elec_4x5.4
- J3, J4, J5, J6: moved to F.Cu
- L1, L2: value FAUL1360-3R3MT -> FAUL1340-3R3MT; footprint Inductor_SMD:L_Bourns_SRR1260 -> Inductor_SMD:L_TechFuse_SL1250
- R18: footprint Capacitor_SMD:C_0805_2012Metric -> Resistor_SMD:R_0805_2012Metric
- RN1, RN2, RN3, RN4, RN5, RN6: footprint Resistor_THT:R_Array_SIP9 -> Package_SIP:SIP-9_22.3x3mm_P2.54mm
- TP1, TP2, TP3, TP4, TP5, TP6, TP7, TP8, TP9: footprint TestPoint:TestPoint_Loop_D1.80mm_Drill1.0mm_Beaded -> TestPoint:TestPoint_Pad_1.5x1.5mm
- U1, U2, U3, U4, U6, U7: footprint Package_SO:SOIC-16_3.9x9.9mm_P1.27mm -> Package_SO:TSSOP-16_4.4x5mm_P0.65mm
- U10, U11: footprint Package_SO:SOIC-18W_7.5x11.6mm_P1.27mm -> Package_SO:SOIC-20W_7.5x12.8mm_P1.27mm
- moved J5 55.6 mm to (273.1, 19.9)
- moved J4 45.8 mm to (274.2, 151.3)
- moved C64 24.6 mm to (248.5, 135.2)
- moved J6 23.4 mm to (273.5, 117.1)
- moved D4 22.6 mm to (115.2, 110.2), turned to 90 degrees
- moved RN2 22.4 mm to (229.7, 147.1), turned to -90 degrees
- moved RN1 20.8 mm to (227.7, 178.3), turned to -90 degrees
- moved J3 20.2 mm to (272.7, 85.2)
- moved RN4 18.1 mm to (230.0, 116.3), turned to -90 degrees
- moved C53 17.1 mm to (215.9, 166.5)
- moved C52 16.7 mm to (215.9, 195.5)
- moved U5 16.6 mm to (248.5, 165.7)
- moved R9 16.3 mm to (103.8, 126.5)
- moved U16 16.1 mm to (249.2, 193.3)
- moved U23 14.7 mm to (248.8, 130.4)
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Connections:
- net /1 Plyr Move Down renamed Net-(J5-Pin_4)
- net /1 Plyr Move Left renamed Net-(J5-Pin_1)
- net /1 Plyr Move Right renamed Net-(J5-Pin_2)
- net /1 Plyr Move Up renamed Net-(J5-Pin_3)
Routing:
- net GND: track 323.8 -> 1391.2 mm, vias 45 -> 71
- net +5V: track 307.4 -> 585.1 mm
- net Out_Latch: track 144.3 -> 181.4 mm
- net J6_Input_Stream: track 177.2 -> 212.4 mm, vias 5 -> 3
- net +3.3V: track 586.2 -> 553.5 mm, vias 13 -> 19
- net Out_Clock: track 150.0 -> 181.5 mm
- net Net-(RN1-R2): track 83.9 -> 58.0 mm, vias 3 -> 1
- net VID_G2: track 135.1 -> 111.4 mm, vias 1 -> 2
- net +12V: track 408.0 -> 385.9 mm, vias 2 -> 6
- net Net-(RN1-R1): track 65.9 -> 87.5 mm, vias 3 -> 1
- net Net-(RN10-R3.2): track 70.0 -> 49.0 mm, vias 1 -> 0
- net Net-(D4-K): track 10.9 -> 31.6 mm
- net Net-(J2_RGBS_Out1-Pin_8): track 97.6 -> 77.2 mm, vias 1 -> 2
- net Out_En_N: track 145.8 -> 164.8 mm, vias 3 -> 4
- net IN_LOAD_N: track 339.2 -> 320.8 mm
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- added copper zone on B.Cu, net GND
- removed copper zone on In2.Cu, net +5V
- removed copper zone on In1.Cu, net GND
