File: MCR_prototype_PCB/control_input_j5.kicad_sch (KiCad schematic)
At the start: 34 parts, among them J5 Conn_01x23_Pin, U3 74AHC165

Commit message: Add files via upload
Parts:
- C25, C26, C27, C28, C29, C30, C31, C32: footprint (none) -> Capacitor_SMD:C_0805_2012Metric; KiLib_Generator (none) -> SMD_2terminal_chip_molded
- D19, D20, D21, D22, D23, D24, D25, D26: KiLib_Generator (none) -> package/gullwing
- J5: footprint (none) -> Connector_PinHeader_2.54mm:PinHeader_1x23_P2.54mm_Horizontal; KiLib_Generator (none) -> connector/pin_header_socket
- R44, R45, R46, R47, R48, R49, R50, R51, R52, R53, R54, R55, R56, R57, R58, R59: footprint (none) -> Resistor_SMD:R_0805_2012Metric; KiLib_Generator (none) -> SMD_2terminal_chip_molded
- U3: footprint (none) -> Package_SO:SOIC-16_3.9x9.9mm_P1.27mm; KiLib_Generator (none) -> package/gullwing
Connections:
- net +5V: now also D19.2 (K), D20.2 (K), D21.2 (K), D22.2 (K), D23.2 (K), D24.2 (K), D25.2 (K), D26.2 (K)
- net GND: no longer D19.2 (K), D20.2 (K), D21.2 (K), D22.2 (K), D23.2 (K), D24.2 (K), D25.2 (K), D26.2 (K)

Commit message: Updated 8/22/26
Parts:
- removed D19, D20, D21, D22, D23, D24, D25, D26: BAT54S, Package_TO_SOT_SMD:SOT-23, symbol Diode:BAT54S
- removed R44, R46, R48, R50, R52, R54, R56, R58: 1k, Resistor_SMD:R_0805_2012Metric, symbol Device:R_Small_US
- removed R45, R47, R49, R51, R53, R55, R57, R59: 4.7k, Resistor_SMD:R_0805_2012Metric, symbol Device:R_Small_US
- added RN11, RN12: 1K Ohm, Resistor_SMD:R_Array_Convex_4x0603, symbol Device:R_Pack04
- added RN3: 4.7k ohm, Resistor_THT:R_Array_SIP9, symbol Device:R_Network08_US
- added U18, U19: SRV05-4, Package_TO_SOT_SMD:SOT-23-6, symbol Power_Protection:SRV05-4
Connections:
- net +5V: now also RN3.1 (common), U18.5 (VP), U19.5 (VP)
- net GND: now also U18.2 (VN), U19.2 (VN)
- net at C28.1, U3.3 (D4): now also RN11.8 (R1.2), RN3.5 (R4)
- net at C28.2: now also U18.6 (IO4)
- net at C25.1, U3.6 (D7): now also RN11.5 (R4.2), RN3.2 (R1)
- net at C25.2: now also U18.3 (IO2)
- net at C26.1, U3.5 (D6): now also RN11.6 (R3.2), RN3.3 (R2)
- net at C29.1, U3.14 (D3): now also RN12.5 (R4.2), RN3.6 (R5)
- net at C29.2: now also U19.3 (IO2)
- net at C32.2: now also U19.6 (IO4)
- net at C31.1, U3.12 (D1): now also RN12.7 (R2.2), RN3.8 (R7)
- net at C31.2: now also U19.4 (IO3)
- net at C27.2: now also U18.4 (IO3)
- net at C26.2: now also U18.1 (IO1)
- net at J5.2 (Pin_2): now also RN12.2 (R2.1)
- net at C32.1, U3.11 (D0): now also RN12.8 (R1.2), RN3.9 (R8)
- net at C27.1, U3.4 (D5): now also RN11.7 (R2.2), RN3.4 (R3)
- net at J5.6 (Pin_6): now also RN11.2 (R2.1)
- net at C30.2: now also U19.1 (IO1)
- net at C30.1, U3.13 (D2): now also RN12.6 (R3.2), RN3.7 (R6)
- net at J5.3 (Pin_3): now also RN12.3 (R3.1)
- net at J5.1 (Pin_1): now also RN12.1 (R1.1)
- net at J5.4 (Pin_4): now also RN12.4 (R4.1)
- net at J5.7 (Pin_7): now also RN11.3 (R3.1)
- net at J5.8 (Pin_8): now also RN11.4 (R4.1)
- net at J5.5 (Pin_5): now also RN11.1 (R1.1)

Commit message: Add files via upload
Connections:
- net 1 Plyr Move Left: now reaches J5.1 (Pin_1), RN12.1 (R1.1)
- net 1 Plyr Move Right: now reaches J5.2 (Pin_2), RN12.2 (R2.1)
- net 1 Plyr Move Up: now reaches J5.3 (Pin_3), RN12.3 (R3.1)
- net 1 Plyr Move Down: now reaches J5.4 (Pin_4), RN12.4 (R4.1)
Changed lines of the file:
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@@
+		)
+	)
+	(label "1 Plyr Move Up"
+		(at 26.67 68.58 0)
+		(effects
+			(font
+				(size 1.27 1.27)
+			)
+			(justify left bottom)
+		)
+	)
+	(label "1 Plyr Move Left"
+		(at 26.67 63.5 0)
+		(effects
+			(font
+				(size 1.27 1.27)
+			)
+			(justify left bottom)
+		)
+	)
+	(label "1 Plyr Move Right"
+		(at 26.67 66.04 0)
+		(effects
+			(font
+				(size 1.27 1.27)
+			)
+			(justify left bottom)
+		)
+	)
+	(label "1 Plyr Move Down"
+		(at 26.67 71.12 0)
+		(effects
+			(font
+				(size 1.27 1.27)
+			)
+			(justify left bottom)
 		)
 	)

Commit message: Add files via upload
Parts:
- removed C25, C26, C27, C28, C29, C30, C31, C32: 0.01 uF, Capacitor_SMD:C_0805_2012Metric, symbol Device:C_Small_US
- added C54, C61, C62: 0.1 uF, Capacitor_SMD:C_0805_2012Metric, symbol Device:C_Small
Connections:
- net +3.3V: now also C54.1
- net +5V: now also C61.2, C62.2
- net GND: now also J5.18 (Pin_18), J5.9 (Pin_9), C54.2, C61.1, C62.1
- net at RN11.5 (R4.2), RN3.2 (R1), U3.6 (D7): now also U18.3 (IO2)
- net at RN12.5 (R4.2), RN3.6 (R5), U3.14 (D3): now also U19.3 (IO2)
- net at RN12.7 (R2.2), RN3.8 (R7), U3.12 (D1): now also U19.4 (IO3)
- net at RN11.6 (R3.2), RN3.3 (R2), U3.5 (D6): now also U18.1 (IO1)
- net at RN11.7 (R2.2), RN3.4 (R3), U3.4 (D5): now also U18.4 (IO3)
- net at RN11.8 (R1.2), RN3.5 (R4), U3.3 (D4): now also U18.6 (IO4)
- net at RN12.6 (R3.2), RN3.7 (R6), U3.13 (D2): now also U19.1 (IO1)
- net at RN12.8 (R1.2), RN3.9 (R8), U3.11 (D0): now also U19.6 (IO4)
- net Coin_Meter_Return renamed +12V
- no-connect marks 6 -> 4

Commit message: Add files via upload
Connections:
- net +12V: now also J5.20 (Pin_20); no longer J5.21 (Pin_21)
- net Coin_Meter: now also J5.21 (Pin_21); no longer J5.20 (Pin_20)
Changed lines of the file:
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@@
+	(wire
+		(pts
+			(xy 62.23 114.3) (xy 38.1 114.3)
+		)
+		(stroke
+			(width 0)
+			(type default)
+		)
+	)
 	(wire
 		(pts
@@
 	(wire
 		(pts
+			(xy 38.1 114.3) (xy 38.1 111.76)
+		)
+		(stroke
+			(width 0)
+			(type default)
+		)
+	)
+	(wire
+		(pts
 			(xy 264.16 138.43) (xy 270.51 138.43)
 		)
@@
 	(wire
 		(pts
+			(xy 38.1 111.76) (xy 24.13 111.76)
+		)
+		(stroke
+			(width 0)
+			(type default)
+		)
+	)
+	(wire
+		(pts
 			(xy 96.52 41.91) (xy 96.52 91.44)
 		)
@@
 	(wire
 		(pts
+			(xy 24.13 114.3) (xy 34.29 114.3)
+		)
+		(stroke
+			(width 0)
+			(type default)
+		)
+	)
+	(wire
+		(pts
 			(xy 24.13 88.9) (xy 27.94 88.9)
 		)
@@
 	(wire
 		(pts
+			(xy 34.29 114.3) (xy 34.29 118.11)
+		)
+		(stroke
+			(width 0)
+			(type default)
+		)
+	)
+	(wire
+		(pts
 			(xy 109.22 41.91) (xy 109.22 71.12)
 		)
@@
 	(wire
 		(pts
-			(xy 24.13 111.76) (xy 31.75 111.76)
-		)
-		(stroke
-			(width 0)
-			(type default)
-		)
-	)
-	(wire
-		(pts
 			(xy 261.62 33.02) (xy 96.52 33.02)
 		)
@@
 		(pts
 			(xy 257.81 109.22) (xy 257.81 67.31)
-		)
-		(stroke
-			(width 0)
-			(type default)
-		)
-	)
-	(wire
-		(pts
-			(xy 24.13 114.3) (xy 62.23 114.3)
 		)
 		(stroke
@@
 	(global_label "Coin_Meter"
 		(shape output)
-		(at 31.75 111.76 0)
+		(at 34.29 118.11 0)
 		(fields_autoplaced yes)
 		(effects
@@
 		)
 		(property "Intersheetrefs" "${INTERSHEET_REFS}"
-			(at 45.0161 111.76 0)
+			(at 47.5561 118.11 0)
 			(hide yes)
 			(show_name no)

Commit message: Production/schematics for 10/10/26 first board run
Parts:
- C54, C61, C62: LCSC (none) -> C49678
- RN11, RN12: LCSC (none) -> C110021
- RN3: footprint Resistor_THT:R_Array_SIP9 -> Package_SIP:SIP-9_22.3x3mm_P2.54mm; LCSC (none) -> C9112
- U18, U19: LCSC (none) -> C558418
- U3: footprint Package_SO:SOIC-16_3.9x9.9mm_P1.27mm -> Package_SO:TSSOP-16_4.4x5mm_P0.65mm; LCSC (none) -> C32498669
Connections:
- net 1 Plyr Move Down: no longer names the net of J5.4 (Pin_4), RN12.4 (R4.1)
- net 1 Plyr Move Left: no longer names the net of J5.1 (Pin_1), RN12.1 (R1.1)
- net 1 Plyr Move Right: no longer names the net of J5.2 (Pin_2), RN12.2 (R2.1)
- net 1 Plyr Move Up: no longer names the net of J5.3 (Pin_3), RN12.3 (R3.1)
