File: MCR_prototype_PCB/control_inputs.kicad_sch (KiCad schematic)
At the start: 67 parts, among them J4 Conn_01x19_Pin, U1 74AHC165, U2 74AHC165

Commit message: Add files via upload
Parts:
- C10, C11, C12, C13, C14, C15, C16, C17, C18, C19, C20, C21, C22, C23, C24, C9: footprint (none) -> Capacitor_SMD:C_0805_2012Metric; KiLib_Generator (none) -> SMD_2terminal_chip_molded
- D10, D11, D12, D13, D14, D15, D16, D17, D18, D3, D4, D5, D6, D7, D8, D9: KiLib_Generator (none) -> package/gullwing
- J4: footprint (none) -> Connector_PinHeader_2.54mm:PinHeader_1x19_P2.54mm_Horizontal; KiLib_Generator (none) -> connector/pin_header_socket
- R12, R13, R14, R15, R16, R17, R18, R19, R20, R21, R22, R23, R24, R25, R26, R27, R28, R29, R30, R31, R32, R33, R34, R35, R36, R37, R38, R39, R40, R41, R42, R43: footprint (none) -> Resistor_SMD:R_0805_2012Metric; KiLib_Generator (none) -> SMD_2terminal_chip_molded
- U1, U2: footprint (none) -> Package_SO:SOIC-16_3.9x9.9mm_P1.27mm; KiLib_Generator (none) -> package/gullwing
Connections:
- net +5V: now also D10.2 (K), D11.2 (K), D12.2 (K), D13.2 (K), D14.2 (K), D15.2 (K), D16.2 (K), D17.2 (K), D18.2 (K), D3.2 (K), D4.2 (K), D5.2 (K), D6.2 (K), D7.2 (K), D8.2 (K), D9.2 (K)
- net GND: no longer D10.2 (K), D11.2 (K), D12.2 (K), D13.2 (K), D14.2 (K), D15.2 (K), D16.2 (K), D17.2 (K), D18.2 (K), D3.2 (K), D4.2 (K), D5.2 (K), D6.2 (K), D7.2 (K), D8.2 (K), D9.2 (K)

Commit message: Updated 8/22/26
Parts:
- removed D10, D11, D12, D13, D14, D15, D16, D17, D18, D3, D4, D5, D6, D7, D8, D9: BAT54S, Package_TO_SOT_SMD:SOT-23, symbol Diode:BAT54S
- removed R12, R13, R14, R15, R16, R17, R18, R19, R20, R21, R33, R35, R37, R39, R41, R43: 4.7k, Resistor_SMD:R_0805_2012Metric, symbol Device:R_Small_US
- removed R22, R23, R24, R25, R26, R27, R28, R29, R30, R31, R32, R34, R36, R38, R40, R42: 1k, Resistor_SMD:R_0805_2012Metric, symbol Device:R_Small_US
- added RN1, RN2: 4.7k ohm, Resistor_THT:R_Array_SIP9, symbol Device:R_Network08_US
- added RN10, RN7, RN8, RN9: 1K Ohm, Resistor_SMD:R_Array_Convex_4x0603, symbol Device:R_Pack04
- added U15, U16, U17, U5: SRV05-4, Package_TO_SOT_SMD:SOT-23-6, symbol Power_Protection:SRV05-4
Connections:
- net +5V: now also RN1.1 (common), RN2.1 (common), U15.5 (VP), U16.5 (VP), U17.5 (VP), U5.5 (VP)
- net GND: now also U15.2 (VN), U16.2 (VN), U17.2 (VN), U5.2 (VN)
- net at C15.1, U1.12 (D1): now also RN1.8 (R7), RN7.6 (R3.2)
- net at C15.2: now also U17.4 (IO3)
- net at C18.2: now also U15.1 (IO1)
- net at C17.1, U2.6 (D7): now also RN2.2 (R1), RN9.5 (R4.2)
- net at J4.18 (Pin_18): now also RN9.4 (R4.1)
- net at C23.1, U2.12 (D1): now also RN10.7 (R2.2), RN2.8 (R7)
- net at J4.11 (Pin_11): now also RN10.2 (R2.1)
- net at C18.1, U2.5 (D6): now also RN2.3 (R2), RN9.6 (R3.2)
- net at C16.1, U1.11 (D0): now also RN1.9 (R8), RN7.5 (R4.2)
- net at C16.2: now also U17.6 (IO4)
- net at C10.1, U1.5 (D6): now also RN1.3 (R2), RN8.6 (R3.2)
- net at C10.2: now also U16.1 (IO1)
- net at C13.1, U1.14 (D3): now also RN1.6 (R5), RN7.8 (R1.2)
- net at J4.5 (Pin_5): now also RN7.1 (R1.1)
- net at J4.8 (Pin_8): now also RN7.4 (R4.1)
- net at C24.1, U2.11 (D0): now also RN10.8 (R1.2), RN2.9 (R8)
- net at C22.1, U2.13 (D2): now also RN10.6 (R3.2), RN2.7 (R6)
- net at C21.1, U2.14 (D3): now also RN10.5 (R4.2), RN2.6 (R5)
- net at C20.1, U2.3 (D4): now also RN2.5 (R4), RN9.8 (R1.2)
- net at C19.1, U2.4 (D5): now also RN2.4 (R3), RN9.7 (R2.2)
- net at J4.13 (Pin_13): now also RN10.4 (R4.1)
- net at J4.16 (Pin_16): now also RN9.2 (R2.1)
- net at C12.1, U1.3 (D4): now also RN1.5 (R4), RN8.8 (R1.2)
- net at C12.2: now also U16.6 (IO4)
- net at C9.2: now also U16.3 (IO2)
- net at C17.2: now also U15.3 (IO2)
- net at C20.2: now also U15.6 (IO4)
- net at J4.2 (Pin_2): now also RN8.3 (R3.1)
- net at C11.1, U1.4 (D5): now also RN1.4 (R3), RN8.7 (R2.2)
- net at J4.3 (Pin_3): now also RN8.2 (R2.1)
- net at C19.2: now also U15.4 (IO3)
- net at J4.10 (Pin_10): now also RN10.1 (R1.1)
- net at C11.2: now also U16.4 (IO3)
- net at C9.1, U1.6 (D7): now also RN1.2 (R1), RN8.5 (R4.2)
- net at C24.2: now also U5.6 (IO4)
- net at C14.2: now also U17.1 (IO1)
- net at J4.17 (Pin_17): now also RN9.3 (R3.1)
- net at C14.1, U1.13 (D2): now also RN1.7 (R6), RN7.7 (R2.2)
- net at J4.7 (Pin_7): now also RN7.3 (R3.1)
- net at C21.2: now also U5.3 (IO2)
- net at J4.1 (Pin_1): now also RN8.4 (R4.1)
- net at J4.12 (Pin_12): now also RN10.3 (R3.1)
- net at J4.15 (Pin_15): now also RN9.1 (R1.1)
- net at J4.4 (Pin_4): now also RN8.1 (R1.1)
- net at J4.6 (Pin_6): now also RN7.2 (R2.1)
- net at C23.2: now also U5.4 (IO3)
- net at C13.2: now also U17.3 (IO2)
- net at C22.2: now also U5.1 (IO1)
Other:
- moved on the sheet: J4, U2

Commit message: Add files via upload
Connections:
- net GND: now also J4.19 (Pin_19), J4.9 (Pin_9)
- no-connect marks 5 -> 3
Changed lines of the file:
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@@
 	)
 	(junction
+		(at 21.59 90.17)
+		(diameter 0)
+		(color 0 0 0 0)
+	)
+	(junction
 		(at 121.92 118.11)
 		(diameter 0)
@@
 	)
 	(no_connect
-		(at 19.05 64.77)
-	)
-	(no_connect
 		(at 262.89 93.98)
 	)
@@
 		(at 19.05 77.47)
 	)
-	(no_connect
-		(at 19.05 90.17)
-	)
 	(wire
 		(pts
@@
 	(wire
 		(pts
+			(xy 21.59 64.77) (xy 21.59 90.17)
+		)
+		(stroke
+			(width 0)
+			(type default)
+		)
+	)
+	(wire
+		(pts
 			(xy 78.74 39.37) (xy 91.44 39.37)
 		)
@@
 	(wire
 		(pts
+			(xy 19.05 90.17) (xy 21.59 90.17)
+		)
+		(stroke
+			(width 0)
+			(type default)
+		)
+	)
+	(wire
+		(pts
 			(xy 213.36 100.33) (xy 213.36 118.11)
 		)
@@
 	(wire
 		(pts
+			(xy 19.05 64.77) (xy 21.59 64.77)
+		)
+		(stroke
+			(width 0)
+			(type default)
+		)
+	)
+	(wire
+		(pts
 			(xy 256.54 33.02) (xy 256.54 24.13)
 		)
@@
 					(unit 1)
 				)
+			)
+		)
+	)
+	(symbol
+		(lib_id "power:GND")
+		(at 21.59 90.17 0)
+		(unit 1)
+		(body_style 1)
+		(exclude_from_sim no)
+		(in_bom yes)
+		(on_board yes)
+		(in_pos_files yes)
+		(dnp no)
+		(fields_autoplaced yes)
+		(property "Reference" "#PWR019"
+			(at 21.59 96.52 0)
+			(hide yes)
+			(show_name no)
+			(do_not_autoplace no)
+			(effects
+				(font
+					(size 1.27 1.27)
+				)
+			)
+		)
+		(property "Value" "GND"
+			(at 21.59 95.25 0)
+			(show_name no)
+			(do_not_autoplace no)
+			(effects
+				(font
+					(size 1.27 1.27)
+				)
+			)
+		)
+		(property "Footprint" ""
+			(at 21.59 90.17 0)
+			(hide yes)
+			(show_name no)
+			(do_not_autoplace no)
+			(effects
+				(font
+					(size 1.27 1.27)
+				)
+			)
+		)
+		(property "Datasheet" ""
+			(at 21.59 90.17 0)
+			(hide yes)
+			(show_name no)
+			(do_not_autoplace no)
+			(effects
+				(font
+					(size 1.27 1.27)
+				)
+			)
+		)
+		(property "Description" "Power symbol creates a global label with name \"GND\" , ground"
+			(at 21.59 90.17 0)
+			(hide yes)
+			(show_name no)
+			(do_not_autoplace no)
+			(effects
+				(font
+					(size 1.27 1.27)
+				)
+			)
+		)
+		(pin "1"
+		)
+		(instances
+			(project "MCR_prototype_PCB"
+				(path "/558b91ae-1f51-4604-a49b-2a82d580a522"
+					(reference "#PWR019")
+					(unit 1)
+				)

Commit message: Add files via upload
Parts:
- removed C10, C11, C12, C13, C14, C15, C16, C17, C18, C19, C20, C21, C22, C23, C24, C9: 0.01 uF, Capacitor_SMD:C_0805_2012Metric, symbol Device:C_Small_US
- added C52, C53: 0.1 uF, Capacitor_SMD:C_0805_2012Metric, symbol Device:C_Small
Connections:
- net +3.3V: now also C52.1, C53.1
- net GND: now also C52.2, C53.2
- net IN_CLK: now also U1.2 (CP), U2.2 (CP); no longer U1.1 (~{PL}), U2.1 (~{PL})
- net IN_LOAD_N: now also U1.1 (~{PL}), U2.1 (~{PL}); no longer U1.2 (CP), U2.2 (CP)
- net at RN1.8 (R7), RN7.6 (R3.2), U1.12 (D1): now also U17.4 (IO3)
- net at RN2.3 (R2), RN9.6 (R3.2), U2.5 (D6): now also U15.1 (IO1)
- net at RN1.9 (R8), RN7.5 (R4.2), U1.11 (D0): now also U17.6 (IO4)
- net at RN1.3 (R2), RN8.6 (R3.2), U1.5 (D6): now also U16.1 (IO1)
- net at RN10.8 (R1.2), RN2.9 (R8), U2.11 (D0): now also U5.6 (IO4)
- net at RN10.7 (R2.2), RN2.8 (R7), U2.12 (D1): now also U5.4 (IO3)
- net at RN10.6 (R3.2), RN2.7 (R6), U2.13 (D2): now also U5.1 (IO1)
- net at RN10.5 (R4.2), RN2.6 (R5), U2.14 (D3): now also U5.3 (IO2)
- net at RN2.5 (R4), RN9.8 (R1.2), U2.3 (D4): now also U15.6 (IO4)
- net at RN2.4 (R3), RN9.7 (R2.2), U2.4 (D5): now also U15.4 (IO3)
- net at RN2.2 (R1), RN9.5 (R4.2), U2.6 (D7): now also U15.3 (IO2)
- net at RN1.5 (R4), RN8.8 (R1.2), U1.3 (D4): now also U16.6 (IO4)
- net at RN1.2 (R1), RN8.5 (R4.2), U1.6 (D7): now also U16.3 (IO2)
- net at RN1.4 (R3), RN8.7 (R2.2), U1.4 (D5): now also U16.4 (IO3)
- net at RN1.6 (R5), RN7.8 (R1.2), U1.14 (D3): now also U17.3 (IO2)
- net at RN1.7 (R6), RN7.7 (R2.2), U1.13 (D2): now also U17.1 (IO1)

Commit message: Production/schematics for 10/10/26 first board run
Parts:
- added C66, C67, C68, C69: 0.1 uF, Capacitor_SMD:C_0805_2012Metric, symbol Device:C_Small
- C52, C53: LCSC (none) -> C49678
- RN1, RN2: footprint Resistor_THT:R_Array_SIP9 -> Package_SIP:SIP-9_22.3x3mm_P2.54mm; LCSC (none) -> C9112
- RN10, RN7, RN8, RN9: LCSC (none) -> C110021
- U1, U2: footprint Package_SO:SOIC-16_3.9x9.9mm_P1.27mm -> Package_SO:TSSOP-16_4.4x5mm_P0.65mm; LCSC (none) -> C32498669
- U15, U16, U17, U5: LCSC (none) -> C558418
Connections:
- net +5V: now also C66.2, C67.2, C68.2, C69.2
- net GND: now also C66.1, C67.1, C68.1, C69.1
