File: MCR_prototype_PCB/lamp_squeak_output_j5.kicad_sch (KiCad schematic)
At the start: 5 parts, among them U10 ULN2803CDWR, U11 ULN2803CDWR, U8 74HC595, U9 74HC595

Commit message: Add files via upload
Parts:
- R103: footprint (none) -> Resistor_SMD:R_0805_2012Metric; KiLib_Generator (none) -> SMD_2terminal_chip_molded
- U10, U11: footprint (none) -> Package_SO:SOIC-18W_7.5x11.6mm_P1.27mm; KiLib_Generator (none) -> package/gullwing
- U8, U9: footprint (none) -> Package_SO:SOIC-16_3.9x9.9mm_P1.27mm; KiLib_Generator (none) -> package/gullwing
Changed lines of the file:
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@@
 			)
 		)
-		(property "Footprint" ""
+		(property "Footprint" "Package_SO:SOIC-18W_7.5x11.6mm_P1.27mm"
 			(at 101.6 129.54 0)
 			(hide yes)
@@
 		)
 		(property "Description" "Darlington Transistor Arrays, SOIC18/DIP18"
+			(at 100.33 113.03 0)
+			(hide yes)
+			(show_name no)
+			(do_not_autoplace no)
+			(effects
+				(font
+					(size 1.27 1.27)
+				)
+			)
+		)
+		(property "KiLib_Generator" "package/gullwing"
 			(at 100.33 113.03 0)
 			(hide yes)
@@
 			)
 		)
-		(property "Footprint" ""
+		(property "Footprint" "Resistor_SMD:R_0805_2012Metric"
 			(at 34.29 71.12 0)
 			(hide yes)
@@
 		)
 		(property "Description" "Resistor, small US symbol"
+			(at 34.29 71.12 0)
+			(hide yes)
+			(show_name no)
+			(do_not_autoplace no)
+			(effects
+				(font
+					(size 1.27 1.27)
+				)
+			)
+		)
+		(property "KiLib_Generator" "SMD_2terminal_chip_molded"
 			(at 34.29 71.12 0)
 			(hide yes)
@@
 			)
 		)
-		(property "Footprint" ""
+		(property "Footprint" "Package_SO:SOIC-18W_7.5x11.6mm_P1.27mm"
 			(at 100.33 71.12 0)
 			(hide yes)
@@
 		)
 		(property "Description" "Darlington Transistor Arrays, SOIC18/DIP18"
+			(at 99.06 54.61 0)
+			(hide yes)
+			(show_name no)
+			(do_not_autoplace no)
+			(effects
+				(font
+					(size 1.27 1.27)
+				)
+			)
+		)
+		(property "KiLib_Generator" "package/gullwing"
 			(at 99.06 54.61 0)
 			(hide yes)
@@
 			)
 		)
-		(property "Footprint" ""
+		(property "Footprint" "Package_SO:SOIC-16_3.9x9.9mm_P1.27mm"
 			(at 63.5 118.11 0)
 			(hide yes)
@@
 		)
 		(property "Description" "8-bit serial in/out Shift Register 3-State Outputs"
+			(at 63.5 118.11 0)
+			(hide yes)
+			(show_name no)
+			(do_not_autoplace no)
+			(effects
+				(font
+					(size 1.27 1.27)
+				)
+			)
+		)
+		(property "KiLib_Generator" "package/gullwing"
 			(at 63.5 118.11 0)
 			(hide yes)
@@
 			)
 		)
-		(property "Footprint" ""
+		(property "Footprint" "Package_SO:SOIC-16_3.9x9.9mm_P1.27mm"
 			(at 62.23 59.69 0)
 			(hide yes)
@@
 			(at 62.23 59.69 0)
 			(hide yes)
+			(show_name no)
+			(do_not_autoplace no)
+			(effects
+				(font
+					(size 1.27 1.27)
+				)
+			)
+		)
+		(property "KiLib_Generator" "package/gullwing"
+			(at 62.23 59.69 0)
+			(hide yes)

Commit message: Add files via upload
Parts:
- added C58, C60: 0.1 uF, Capacitor_SMD:C_0805_2012Metric, symbol Device:C_Small
- added R104: 10k, Resistor_SMD:R_0805_2012Metric, symbol Device:R_Small_US
Connections:
- net +3.3V: now also R104.1
- net +5V: now also C58.1, C60.1
- net GND: now also C58.2, C60.2
- net Out_Clear: now also R104.2
- net Coin_Meter_Return: no longer names the net of U10.17 (O2)
- no-connect marks 4 -> 5

Commit message: Production/schematics for 10/10/26 first board run
Parts:
- C58, C60: LCSC (none) -> C49678
- R103, R104: LCSC (none) -> C17414
- U10, U11: footprint Package_SO:SOIC-18W_7.5x11.6mm_P1.27mm -> Package_SO:SOIC-20W_7.5x12.8mm_P1.27mm; LCSC (none) -> C7494313
- U8, U9: LCSC (none) -> C18164493
