File: MCR_prototype_PCB/service_switch.kicad_sch (KiCad schematic)
At the start: 2 parts, among them SW4 Service

Commit message: Add files via upload
Parts:
- removed SW4: Service, Button_Switch_SMD:SW_SPDT_CK_JS102011SAQN, symbol Switch:SW_DPDT_x2
- added SW3: Service, Button_Switch_SMD:SW_SPST_PTS645Sx43SMTR92, symbol Switch:SW_Push
Connections:
- net GND: now also SW3.1
- net Service Switch: now also SW3.2
- no-connect marks 4 -> 0
Changed lines of the file:
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@@
 		(color 0 0 0 0)
 	)
-	(no_connect
-		(at 143.51 109.22)
-	)
-	(no_connect
-		(at 133.35 106.68)
-	)
-	(no_connect
-		(at 143.51 85.09)
-	)
-	(no_connect
-		(at 143.51 104.14)
-	)
 	(wire
 		(pts
@@
 		(pts
 			(xy 149.86 85.09) (xy 149.86 90.17)
+		)
+		(stroke
+			(width 0)
+			(type default)
+		)
+	)
+	(wire
+		(pts
+			(xy 143.51 87.63) (xy 143.51 90.17)
 		)
 		(stroke
@@
 	)
 	(symbol
-		(lib_id "Switch:SW_DPDT_x2")
-		(at 138.43 106.68 0)
-		(unit 2)
-		(body_style 1)
-		(exclude_from_sim no)
-		(in_bom yes)
-		(on_board yes)
-		(in_pos_files yes)
-		(dnp no)
-		(fields_autoplaced yes)
-		(property "Reference" "SW4"
-			(at 138.43 97.79 0)
-			(show_name no)
-			(do_not_autoplace no)
-			(effects
-				(font
-					(size 1.27 1.27)
-				)
-			)
-		)
-		(property "Value" "Service"
-			(at 138.43 100.33 0)
-			(show_name no)
-			(do_not_autoplace no)
-			(effects
-				(font
-					(size 1.27 1.27)
-				)
-			)
-		)
-		(property "Footprint" "Button_Switch_SMD:SW_SPDT_CK_JS102011SAQN"
-			(at 138.43 106.68 0)
-			(hide yes)
-			(show_name no)
-			(do_not_autoplace no)
-			(effects
-				(font
-					(size 1.27 1.27)
-				)
-			)
-		)
-		(property "Datasheet" ""
-			(at 138.43 106.68 0)
-			(hide yes)
-			(show_name no)
-			(do_not_autoplace no)
-			(effects
-				(font
-					(size 1.27 1.27)
-				)
-			)
-		)
-		(property "Description" "Switch, dual pole double throw, separate symbols"
-			(at 138.43 106.68 0)
-			(hide yes)
-			(show_name no)
-			(do_not_autoplace no)
-			(effects
-				(font
-					(size 1.27 1.27)
-				)
-			)
-		)
-		(pin "5"
-		)
-		(pin "1"
-		)
-		(pin "2"
-		)
-		(pin "4"
-		)
-		(pin "3"
-		)
-		(pin "6"
-		)
-		(instances
-			(project "MCR_prototype_PCB"
-				(path "/08fc2143-0f49-4309-b36c-73646f69ff7b"
-					(reference "SW4")
-					(unit 2)
-				)
-			)
-		)
-	)
-	(symbol
 		(lib_id "power:GND")
 		(at 124.46 93.98 0)
@@
 	)
 	(symbol
-		(lib_id "Switch:SW_DPDT_x2")
+		(lib_id "Switch:SW_Push")
 		(at 138.43 87.63 0)
 		(unit 1)
@@
 		(dnp no)
 		(fields_autoplaced yes)
-		(property "Reference" "SW4"
-			(at 138.43 78.74 0)
+		(property "Reference" "SW3"
+			(at 138.43 80.01 0)
 			(show_name no)
 			(do_not_autoplace no)
@@
 		)
 		(property "Value" "Service"
-			(at 138.43 81.28 0)
-			(show_name no)
-			(do_not_autoplace no)
-			(effects
-				(font
-					(size 1.27 1.27)
-				)
-			)
-		)
-		(property "Footprint" "Button_Switch_SMD:SW_SPDT_CK_JS102011SAQN"
+			(at 138.43 82.55 0)
+			(show_name no)
+			(do_not_autoplace no)
+			(effects
+				(font
+					(size 1.27 1.27)
+				)
+			)
+		)
+		(property "Footprint" "Button_Switch_SMD:SW_SPST_PTS645Sx43SMTR92"
+			(at 138.43 82.55 0)
+			(hide yes)
+			(show_name no)
+			(do_not_autoplace no)
+			(effects
+				(font
+					(size 1.27 1.27)
+				)
+			)
+		)
+		(property "Datasheet" ""
+			(at 138.43 82.55 0)
+			(hide yes)
+			(show_name no)
+			(do_not_autoplace no)
+			(effects
+				(font
+					(size 1.27 1.27)
+				)
+			)
+		)
+		(property "Description" "Push button switch, generic, two pins"
 			(at 138.43 87.63 0)
 			(hide yes)
@@
 			)
 		)
-		(property "Datasheet" ""
-			(at 138.43 87.63 0)
-			(hide yes)
-			(show_name no)
-			(do_not_autoplace no)
-			(effects
-				(font
-					(size 1.27 1.27)
-				)
-			)
-		)
-		(property "Description" "Switch, dual pole double throw, separate symbols"
-			(at 138.43 87.63 0)
-			(hide yes)
-			(show_name no)
-			(do_not_autoplace no)
-			(effects
-				(font
-					(size 1.27 1.27)
-				)
-			)
-		)
-		(pin "5"
+		(pin "2"
 		)
 		(pin "1"
-		)
-		(pin "2"
-		)
-		(pin "4"
-		)
-		(pin "3"
-		)
-		(pin "6"
 		)
 		(instances
 			(project "MCR_prototype_PCB"
 				(path "/08fc2143-0f49-4309-b36c-73646f69ff7b"
-					(reference "SW4")
+					(reference "SW3")
 					(unit 1)
 				)

Commit message: September 8 Version
Parts:
- SW3: value Service -> PTS645SM43SMTR92LFS; LCSC (none) -> C221880
Changed lines of the file:
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@@
 			)
 		)
-		(property "Value" "Service"
+		(property "Value" "PTS645SM43SMTR92LFS"
 			(at 138.43 82.55 0)
 			(show_name no)
@@
 			(at 138.43 87.63 0)
 			(hide yes)
+			(show_name no)
+			(do_not_autoplace no)
+			(effects
+				(font
+					(size 1.27 1.27)
+				)
+			)
+		)
+		(property "LCSC" "C221880"
+			(at 138.43 87.63 0)
+			(hide yes)

Commit message: Production/schematics for 10/10/26 first board run
Parts:
- R9: LCSC (none) -> C17513
Changed lines of the file:
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@@
+			)
+		)
+		(property "LCSC" "C17513"
+			(at 149.86 82.55 0)
+			(hide yes)
+			(show_name no)
+			(do_not_autoplace no)
+			(effects
+				(font
+					(size 1.27 1.27)
+				)
+			)
+		)
+		(property "KLC_S3.3" ""
+			(at 149.86 82.55 0)
+			(hide yes)
+			(show_name no)
+			(do_not_autoplace no)
+			(effects
+				(font
+					(size 1.27 1.27)
+				)
+			)
+		)
+		(property "KLC_S5.1" ""
+			(at 149.86 82.55 0)
+			(hide yes)
+			(show_name no)
+			(do_not_autoplace no)
+			(effects
+				(font
+					(size 1.27 1.27)
+				)
 			)
 		)
@@
 			(at 138.43 87.63 0)
 			(hide yes)
+			(show_name no)
+			(do_not_autoplace no)
+			(effects
+				(font
+					(size 1.27 1.27)
+				)
+			)
+		)
+		(property "KLC_S3.3" ""
+			(at 138.43 87.63 0)
+			(hide yes)
+			(show_name no)
+			(do_not_autoplace no)
+			(effects
+				(font
+					(size 1.27 1.27)
+				)
+			)
+		)
+		(property "KLC_S5.1" ""
+			(at 138.43 87.63 0)
+			(hide yes)
