File: MCR_prototype_PCB/video_outputs.kicad_sch (KiCad schematic)
At the start: 22 parts, among them J1-VGAOut1 DE15_Socket_HighDensity, J2_CPU1 Conn_01x09_Pin, U12 THS7374, U13 THS7374

Commit message: Add files via upload
Parts:
- C41, C42: footprint (none) -> Capacitor_SMD:C_0805_2012Metric; KiLib_Generator (none) -> SMD_2terminal_chip_molded
- C43, C44: footprint (none) -> Capacitor_SMD:C_1210_3225Metric; KiLib_Generator (none) -> SMD_2terminal_chip_molded
- J1-VGAOut1: footprint (none) -> Connector_Dsub:DSUB-15-HD_Socket_Horizontal_P2.29x1.90mm_EdgePinOffset3.03mm_Housed_MountingHolesOffset4.94mm
- J2_RGBS_Out1: renamed from J2_CPU1; footprint (none) -> Connector_PinHeader_2.54mm:PinHeader_1x09_P2.54mm_Horizontal; KiLib_Generator (none) -> connector/pin_header_socket
- JP1, JP2, JP3: footprint Connector_PinHeader_1.00mm:PinHeader_1x02_P1.00mm_Vertical -> Connector_PinHeader_2.54mm:PinHeader_1x02_P2.54mm_Vertical; KiLib_Generator (none) -> connector/pin_header_socket
- R100, R101, R102, R92, R93, R94, R95, R96, R97, R98, R99: footprint (none) -> Resistor_SMD:R_0805_2012Metric; KiLib_Generator (none) -> SMD_2terminal_chip_molded
- U12, U13: KiLib_Generator (none) -> package/gullwing

Commit message: Updated 8/22/26
Parts:
- R101, R95, R98: value 1000 -> 1k
- R102, R96, R99: value 2000 -> 2k
Changed lines of the file:
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@@
 			)
 		)
-		(property "Value" "2000"
+		(property "Value" "2k"
 			(at 167.64 76.2 90)
 			(show_name no)
@@
 			)
 		)
-		(property "Value" "2000"
+		(property "Value" "2k"
 			(at 167.64 104.14 90)
 			(show_name no)
@@
 			)
 		)
-		(property "Value" "1000"
+		(property "Value" "1k"
 			(at 167.64 124.46 90)
 			(show_name no)
@@
 			)
 		)
-		(property "Value" "1000"
+		(property "Value" "1k"
 			(at 167.64 95.25 90)
 			(show_name no)
@@
 			)
 		)
-		(property "Value" "1000"
+		(property "Value" "1k"
 			(at 167.64 67.31 90)
 			(show_name no)
@@
 			)
 		)
-		(property "Value" "2000"
+		(property "Value" "2k"
 			(at 167.64 133.35 90)
 			(show_name no)

Commit message: Add files via upload
Parts:
- added TP7: VID_HS, TestPoint:TestPoint_Loop_D1.80mm_Drill1.0mm_Beaded, symbol Connector:TestPoint
- added TP8: VID_VS, TestPoint:TestPoint_Loop_D1.80mm_Drill1.0mm_Beaded, symbol Connector:TestPoint
- added TP9: GND, TestPoint:TestPoint_Loop_D1.80mm_Drill1.0mm_Beaded, symbol Connector:TestPoint
Connections:
- net GND: now also TP9.1
- net at J1-VGAOut1.13, J2_RGBS_Out1.8 (Pin_8), U12.14 (CH1_OUT): now also TP7.1
- net at J1-VGAOut1.14, J2_RGBS_Out1.9 (Pin_9), U12.13 (CH2_OUT): now also TP8.1

Commit message: Add files via upload
Parts:
- added JP4: VGA Filter, Connector_PinHeader_2.54mm:PinHeader_1x03_P2.54mm_Vertical, symbol Jumper:Jumper_3_Open
- added R14, R15, R16, R17: 75, Resistor_SMD:R_0805_2012Metric, symbol Device:R_US
- added R18: 75, Capacitor_SMD:C_0805_2012Metric, symbol Device:R_US
Connections:
- net +5V: now also JP4.1 (A)
- net GND: now also JP4.3 (B); no longer U12.9 (BYPASS), U13.9 (BYPASS)
- net at J1-VGAOut1.1, J2_RGBS_Out1.1 (Pin_1): now also R16.2; no longer U13.14 (CH1_OUT)
- net at J1-VGAOut1.2, J2_RGBS_Out1.3 (Pin_3): now also R17.2; no longer U13.12 (CH3_OUT)
- net at J1-VGAOut1.3, J2_RGBS_Out1.5 (Pin_5): now also R18.2; no longer U13.13 (CH2_OUT)
- net at J1-VGAOut1.13, J2_RGBS_Out1.8 (Pin_8), TP7.1: now also R14.2; no longer U12.14 (CH1_OUT)
- net at J1-VGAOut1.14, J2_RGBS_Out1.9 (Pin_9), TP8.1: now also R15.2; no longer U12.13 (CH2_OUT)
- new net: JP4.2 (C), U12.9 (BYPASS), U13.9 (BYPASS)
- new net: R18.1, U13.13 (CH2_OUT)
- new net: R14.1, U12.14 (CH1_OUT)
- new net: R17.1, U13.12 (CH3_OUT)
- new net: R15.1, U12.13 (CH2_OUT)
- new net: R16.1, U13.14 (CH1_OUT)
Other:
- moved on the sheet: J1-VGAOut1, J2_RGBS_Out1, TP7, TP8, TP9

Commit message: Add files via upload
Parts:
- added R19, R20, R21: 75, Resistor_SMD:R_0805_2012Metric, symbol Device:R_US
Connections:
- net GND: now also R19.2, R20.2, R21.2
- net at R100.1, R101.1, R102.1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: now also R21.1
- net at R97.1, R98.1, R99.1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: now also R20.1
- net at R94.1, R95.1, R96.1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: now also R19.1

Commit message: Production/schematics for 10/10/26 first board run
Parts:
- C41, C42: LCSC (none) -> C49678
- C43, C44: LCSC (none) -> C21397
- J1-VGAOut1: LCSC (none) -> C75754
- JP1, JP2, JP3: LCSC (none) -> C492401
- JP4: LCSC (none) -> C2937625; now in the parts list
- R100, R94, R97: LCSC (none) -> C17734
- R101, R95, R98: LCSC (none) -> C17513
- R102, R96, R99: LCSC (none) -> C17604
- R14, R15, R16, R17, R19, R20, R21: LCSC (none) -> C17820
- R18: footprint Capacitor_SMD:C_0805_2012Metric -> Resistor_SMD:R_0805_2012Metric; LCSC (none) -> C17820
- R92, R93: LCSC (none) -> C17408
- TP7, TP8, TP9: footprint TestPoint:TestPoint_Loop_D1.80mm_Drill1.0mm_Beaded -> TestPoint:TestPoint_Pad_1.5x1.5mm
- U12, U13: LCSC (none) -> C2652746
